Commit message: update

File: scout/scout_description/urdf/scout_v2.xacro (robot description, xacro)
@@ -58,4 +58,30 @@
         <child link="inertial_link" />
     </joint>
+     <joint name="hokuyo_joint" type="fixed">
+        <axis xyz="0 1 0" />
+        <origin xyz="0 0 0.4" rpy="0 0 0"/>
+        <parent link="base_link"/>
+        <child link="hokuyo_link"/>
+      </joint>
+      <!-- Hokuyo Laser -->
+      <link name="hokuyo_link">
+        <collision>
+          <origin xyz="0 0 0" rpy="0 0 0"/>
+          <geometry>
+        <box size="0.1 0.1 0.1"/>
+          </geometry>
+        </collision>
+        <visual>
+          <origin xyz="0 0 0" rpy="0 0 0"/>
+          <geometry>
+            <mesh filename="package://scout_description/meshes/hokuyo.dae"/>
+          </geometry>
+        </visual>
+        <inertial>
+          <mass value="1e-5" />
+          <origin xyz="0 0 0" rpy="0 0 0"/>
+          <inertia ixx="1e-6" ixy="0" ixz="0" iyy="1e-6" iyz="0" izz="1e-6" />
+        </inertial>
+      </link>
     <!-- For testing, hang the robot up in the air -->
     <!-- <link name="world" />

Commit message: update

File: scout/scout_description/urdf/scout_v2.xacro (robot description, xacro)
@@ -60,5 +60,5 @@
      <joint name="hokuyo_joint" type="fixed">
         <axis xyz="0 1 0" />
-        <origin xyz="0 0 0.4" rpy="0 0 0"/>
+        <origin xyz="0.0 0 0.2" rpy="0 0 0"/>
         <parent link="base_link"/>
         <child link="hokuyo_link"/>
